Commit message: add new reward

File: src/Balance_Car_RL/assets/data/balboa/balboa.urdf (robot description, URDF)
Before this commit: robot balboa_balancing_robot_kit, 3 links, 2 joints
Links:
- link base_link: geometry collision mesh filename=meshes/body_collision.stl; visual mesh filename=meshes/base_bal01a01_bal01a01.stl
